File: top/vonreg_top.kicad_pcb (KiCad board)
At the start: 2 copper layers, 110 x 81.5 mm, 23 parts, among them K1 SW_Push, K10 SW_Push, K11 SW_Push, K12 SW_Push, K15 SW_Push, K2 SW_Push, K3 SW_Push, K4 SW_Push, K5 SW_Push, K6 SW_Push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

Commit message: V1 ordered PCB
Parts:
- removed HOLE1 (x5): MountingHole_2.5mm_Pad, MountingHole:MountingHole_2.5mm_Pad
- removed M1: MountingHole_2mm, MountingHole:MountingHole_2mm
- added H1: MountingHole_3mm, MountingHole:MountingHole_3mm, F.Cu at (94.0, 93.6)
- added H1: MountingHole_3mm, MountingHole:MountingHole_3mm, F.Cu at (153.3, 90.0)
- added H1: MountingHole_3mm, MountingHole:MountingHole_3mm, F.Cu at (93.9, 73.4)
- added H1: MountingHole_3mm, MountingHole:MountingHole_3mm, F.Cu at (113.2, 88.8)
- added H1: MountingHole_3mm, MountingHole:MountingHole_3mm, F.Cu at (134.4, 59.4)
Changed lines of the file:
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@@
   )
   (paper "A4")
+  (title_block
+    (title "Vonreg Top")
+    (date "2022-03-19")
+    (rev "1.0")
+    (company "Appman")
+  )
   (layers
     (0 "F.Cu" signal)
@@
       (net 12 "/RT9") (pinfunction "2") (pintype "passive"))
   )
-  (footprint "MountingHole:MountingHole_2mm" (layer "F.Cu")
-    (at 113.411 88.519)
-    (descr "Mounting Hole 2mm, no annular")
-    (tags "mounting hole 2mm no annular")
+  (footprint "MountingHole:MountingHole_3mm" (layer "F.Cu")
+    (at 93.98 93.599)
+    (descr "Mounting Hole 3mm, no annular")
+    (tags "mounting hole 3mm no annular")
     (attr exclude_from_pos_files exclude_from_bom)
-    (fp_text reference "M1" (at 0 -3.2) (layer "F.SilkS") hide
-      (effects (font (size 1 1) (thickness 0.15)))
-    )
-    (fp_text value "MountingHole_2mm" (at 0 3.1) (layer "F.Fab") hide
+    (fp_text reference "H1" (at 0 -4) (layer "F.SilkS") hide
+      (effects (font (size 1 1) (thickness 0.15)))
+    )
+    (fp_text value "MountingHole_3mm" (at 0 4) (layer "F.Fab") hide
       (effects (font (size 1 1) (thickness 0.15)))
     )
@@
       (effects (font (size 1 1) (thickness 0.15)))
     )
-    (fp_circle (center 0 0) (end 2 0) (layer "Cmts.User") (width 0.15) (fill none))
-    (fp_circle (center 0 0) (end 2.25 0) (layer "F.CrtYd") (width 0.05) (fill none))
-    (pad "" np_thru_hole circle (at 0 0) (size 2 2) (drill 2) (layers *.Cu *.Mask))
+    (fp_circle (center 0 0) (end 3 0) (layer "Cmts.User") (width 0.15) (fill none))
+    (fp_circle (center 0 0) (end 3.25 0) (layer "F.CrtYd") (width 0.05) (fill none))
+    (pad "" np_thru_hole circle (at 0 0) (size 3 3) (drill 3) (layers *.Cu *.Mask))
   )
   (footprint "Button_Switch_Keyboard:Kailh_socket_MX_optional_reversible" (layer "F.Cu")
@@
       (net 9 "/RT6") (pinfunction "2") (pintype "passive"))
   )
-  (footprint "MountingHole:MountingHole_2.5mm_Pad" (layer "F.Cu")
-    (at 136.144 70.612)
-    (descr "Mounting Hole 2.5mm")
-    (tags "mounting hole 2.5mm")
-    (attr exclude_from_pos_files exclude_from_bom)
-    (fp_text reference "HOLE1" (at 0 -3.5) (layer "F.SilkS") hide
-      (effects (font (size 1 1) (thickness 0.15)))
-    )
-    (fp_text value "MountingHole_2.5mm_Pad" (at 0 3.5) (layer "F.Fab") hide
-      (effects (font (size 1 1) (thickness 0.15)))
-    )
-    (fp_text user "${REFERENCE}" (at 0.3 0) (layer "F.Fab") hide
-      (effects (font (size 1 1) (thickness 0.15)))
-    )
-    (fp_circle (center 0 0) (end 2.5 0) (layer "Cmts.User") (width 0.15) (fill none))
-    (fp_circle (center 0 0) (end 2.75 0) (layer "F.CrtYd") (width 0.05) (fill none))
-    (pad "1" thru_hole circle (at 0 0) (size 5 5) (drill 2.5) (layers *.Cu *.Mask))
-  )
-  (footprint "MountingHole:MountingHole_2.5mm_Pad" (layer "F.Cu")
-    (at 136.017 90.678)
-    (descr "Mounting Hole 2.5mm")
-    (tags "mounting hole 2.5mm")
-    (attr exclude_from_pos_files exclude_from_bom)
-    (fp_text reference "HOLE1" (at 0 -3.5) (layer "F.SilkS") hide
-      (effects (font (size 1 1) (thickness 0.15)))
-    )
-    (fp_text value "MountingHole_2.5mm_Pad" (at 0 3.5) (layer "F.Fab") hide
-      (effects (font (size 1 1) (thickness 0.15)))
-    )
-    (fp_text user "${REFERENCE}" (at 0.3 0) (layer "F.Fab") hide
-      (effects (font (size 1 1) (thickness 0.15)))
-    )
-    (fp_circle (center 0 0) (end 2.5 0) (layer "Cmts.User") (width 0.15) (fill none))
-    (fp_circle (center 0 0) (end 2.75 0) (layer "F.CrtYd") (width 0.05) (fill none))
-    (pad "1" thru_hole circle (at 0 0) (size 5 5) (drill 2.5) (layers *.Cu *.Mask))
-  )
   (footprint "Button_Switch_Keyboard:Kailh_socket_MX_optional_reversible" (layer "F.Cu")
     (at 144.3355 80.264)
@@
       (net 14 "/RT11") (pinfunction "2") (pintype "passive"))
   )
-  (footprint "MountingHole:MountingHole_2.5mm_Pad" (layer "F.Cu")
-    (at 153.797 89.027)
-    (descr "Mounting Hole 2.5mm")
-    (tags "mounting hole 2.5mm")
+  (footprint "MountingHole:MountingHole_3mm" (layer "F.Cu")
+    (at 153.289 90.043)
+    (descr "Mounting Hole 3mm, no annular")
+    (tags "mounting hole 3mm no annular")
     (attr exclude_from_pos_files exclude_from_bom)
-    (fp_text reference "HOLE1" (at 0 -3.5) (layer "F.SilkS") hide
-      (effects (font (size 1 1) (thickness 0.15)))
-    )
-    (fp_text value "MountingHole_2.5mm_Pad" (at 0 3.5) (layer "F.Fab") hide
+    (fp_text reference "H1" (at 0 -4) (layer "F.SilkS") hide
+      (effects (font (size 1 1) (thickness 0.15)))
+    )
+    (fp_text value "MountingHole_3mm" (at 0 4) (layer "F.Fab") hide
       (effects (font (size 1 1) (thickness 0.15)))
     )
@@
       (effects (font (size 1 1) (thickness 0.15)))
     )
-    (fp_circle (center 0 0) (end 2.5 0) (layer "Cmts.User") (width 0.15) (fill none))
-    (fp_circle (center 0 0) (end 2.75 0) (layer "F.CrtYd") (width 0.05) (fill none))
-    (pad "1" thru_hole circle (at 0 0) (size 5 5) (drill 2.5) (layers *.Cu *.Mask))
+    (fp_circle (center 0 0) (end 3 0) (layer "Cmts.User") (width 0.15) (fill none))
+    (fp_circle (center 0 0) (end 3.25 0) (layer "F.CrtYd") (width 0.05) (fill none))
+    (pad "" np_thru_hole circle (at 0 0) (size 3 3) (drill 3) (layers *.Cu *.Mask))
   )
   (footprint "Connector_PinHeader_2.54mm:PinHeader_2x05_P2.54mm_Vertical" (layer "F.Cu")
@@
       (net 10 "/RT7") (pinfunction "2") (pintype "passive"))
   )
-  (footprint "MountingHole:MountingHole_2.5mm_Pad" (layer "F.Cu")
-    (at 93.98 73.152)
-    (descr "Mounting Hole 2.5mm")
-    (tags "mounting hole 2.5mm")
+  (footprint "MountingHole:MountingHole_3mm" (layer "F.Cu")
+    (at 93.853 73.406)
+    (descr "Mounting Hole 3mm, no annular")
+    (tags "mounting hole 3mm no annular")
     (attr exclude_from_pos_files exclude_from_bom)
-    (fp_text reference "HOLE1" (at 0 -3.5) (layer "F.SilkS") hide
-      (effects (font (size 1 1) (thickness 0.15)))
-    )
-    (fp_text value "MountingHole_2.5mm_Pad" (at 0 3.5) (layer "F.Fab") hide
+    (fp_text reference "H1" (at 0 -4) (layer "F.SilkS") hide
+      (effects (font (size 1 1) (thickness 0.15)))
+    )
+    (fp_text value "MountingHole_3mm" (at 0 4) (layer "F.Fab") hide
       (effects (font (size 1 1) (thickness 0.15)))
     )
@@
       (effects (font (size 1 1) (thickness 0.15)))
     )
-    (fp_circle (center 0 0) (end 2.5 0) (layer "Cmts.User") (width 0.15) (fill none))
-    (fp_circle (center 0 0) (end 2.75 0) (layer "F.CrtYd") (width 0.05) (fill none))
-    (pad "1" thru_hole circle (at 0 0) (size 5 5) (drill 2.5) (layers *.Cu *.Mask))
-  )
-  (footprint "MountingHole:MountingHole_2.5mm_Pad" (layer "F.Cu")
-    (at 93.853 93.472)
-    (descr "Mounting Hole 2.5mm")
-    (tags "mounting hole 2.5mm")
+    (fp_circle (center 0 0) (end 3 0) (layer "Cmts.User") (width 0.15) (fill none))
+    (fp_circle (center 0 0) (end 3.25 0) (layer "F.CrtYd") (width 0.05) (fill none))
+    (pad "" np_thru_hole circle (at 0 0) (size 3 3) (drill 3) (layers *.Cu *.Mask))
+  )
+  (footprint "MountingHole:MountingHole_3mm" (layer "F.Cu")
+    (at 113.157 88.773)
+    (descr "Mounting Hole 3mm, no annular")
+    (tags "mounting hole 3mm no annular")
     (attr exclude_from_pos_files exclude_from_bom)
-    (fp_text reference "HOLE1" (at 0 -3.5) (layer "F.SilkS") hide
-      (effects (font (size 1 1) (thickness 0.15)))
-    )
-    (fp_text value "MountingHole_2.5mm_Pad" (at 0 3.5) (layer "F.Fab") hide
+    (fp_text reference "H1" (at 0 -4) (layer "F.SilkS") hide
+      (effects (font (size 1 1) (thickness 0.15)))
+    )
+    (fp_text value "MountingHole_3mm" (at 0 4) (layer "F.Fab") hide
       (effects (font (size 1 1) (thickness 0.15)))
     )
@@
       (effects (font (size 1 1) (thickness 0.15)))
     )
-    (fp_circle (center 0 0) (end 2.5 0) (layer "Cmts.User") (width 0.15) (fill none))
-    (fp_circle (center 0 0) (end 2.75 0) (layer "F.CrtYd") (width 0.05) (fill none))
-    (pad "1" thru_hole circle (at 0 0) (size 5 5) (drill 2.5) (layers *.Cu *.Mask))
+    (fp_circle (center 0 0) (end 3 0) (layer "Cmts.User") (width 0.15) (fill none))
+    (fp_circle (center 0 0) (end 3.25 0) (layer "F.CrtYd") (width 0.05) (fill none))
+    (pad "" np_thru_hole circle (at 0 0) (size 3 3) (drill 3) (layers *.Cu *.Mask))
   )
   (footprint "Connector_PinHeader_2.54mm:PinHeader_2x05_P2.54mm_Vertical" (layer "F.Cu")
@@
       (net 4 "/RT2") (pinfunction "2") (pintype "passive"))
   )
+  (footprint "MountingHole:MountingHole_3mm" (layer "F.Cu")
+    (at 134.366 59.436)
+    (descr "Mounting Hole 3mm, no annular")
+    (tags "mounting hole 3mm no annular")
+    (attr exclude_from_pos_files exclude_from_bom)
+    (fp_text reference "H1" (at 0 -4) (layer "F.SilkS") hide
+      (effects (font (size 1 1) (thickness 0.15)))
+    )
+    (fp_text value "MountingHole_3mm" (at 0 4) (layer "F.Fab") hide
+      (effects (font (size 1 1) (thickness 0.15)))
+    )
+    (fp_text user "${REFERENCE}" (at 0.3 0) (layer "F.Fab") hide
+      (effects (font (size 1 1) (thickness 0.15)))
+    )
+    (fp_circle (center 0 0) (end 3 0) (layer "Cmts.User") (width 0.15) (fill none))
+    (fp_circle (center 0 0) (end 3.25 0) (layer "F.CrtYd") (width 0.05) (fill none))
+    (pad "" np_thru_hole circle (at 0 0) (size 3 3) (drill 3) (layers *.Cu *.Mask))
+  )
   (footprint "Button_Switch_Keyboard:Kailh_socket_MX_optional_reversible" (layer "F.Cu")
